File: STM32NGFF.kicad_pcb (KiCad board)
At the start: 2 copper layers, 32.8 x 70 mm, 26 parts, among them J1 2199119-4, P1 CX70M-24P1, U1 STM32F303CCTx, U2 USBLC6-2SC6, Y1 16MHz

Commit message: added github repo to schematic and PCB
Parts:
- removed C1: 4u7, Capacitor_SMD:C_0603_1608Metric
- removed C2, C3, C4, C5: 100n, Capacitor_SMD:C_0201_0603Metric
- removed C6: 1u, Capacitor_SMD:C_0402_1005Metric
- removed C7: 10n, Capacitor_SMD:C_0603_1608Metric
- removed C8, C9: 12p, Capacitor_SMD:C_0402_1005Metric
- removed D1: RED, LED_SMD:LED_0603_1608Metric
- removed D2: GREEN, LED_SMD:LED_0603_1608Metric
- removed H1: MountingHole_Pad, MountingHole:MountingHole_2.2mm_M2_Pad_Via
- removed J1: 2199119-4, TE:TE_2199119-4
- removed L1: 39n, Inductor_SMD:L_0402_1005Metric
- removed P1: CX70M-24P1, CX70M-24P1:HRS_CX70M-24P1
- removed R1: 2k, Resistor_SMD:R_0603_1608Metric
- removed R10, R9: 5.11k, Resistor_SMD:R_0402_1005Metric
- removed R2, R7: 1k, Resistor_SMD:R_0603_1608Metric
- removed R3: 10k, Resistor_SMD:R_0402_1005Metric
- removed R4: 47, Resistor_SMD:R_0402_1005Metric
- removed R8: 1k5, Resistor_SMD:R_0603_1608Metric
- removed U1: STM32F303CCTx, Package_QFP:LQFP-48_7x7mm_P0.5mm
- removed U2: USBLC6-2SC6, Package_TO_SOT_SMD:SOT-23-6
- removed Y1: 16MHz, Crystal:Crystal_SMD_3225-4Pin_3.2x2.5mm
Routing:
- net +3V3: track 8.57 -> 0.00 mm
Other:
- board outline removed
