File: STM32NGFF.kicad_pcb (KiCad board)
At the start: 2 copper layers, 0 parts

Commit message: Added initial PCB, and updated all global labels to net labels
Parts:
- added C1: 12p, Capacitor_SMD:C_0603_1608Metric, F.Cu at (168.0, 134.2)
- added C10: 100n, Capacitor_SMD:C_0603_1608Metric, F.Cu at (147.3, 148.3)
- added C11: 1u, Capacitor_SMD:C_0603_1608Metric, F.Cu at (143.3, 148.3)
- added C12: 10n, Capacitor_SMD:C_0603_1608Metric, F.Cu at (165.9, 137.7)
- added C2: 12p, Capacitor_SMD:C_0603_1608Metric, F.Cu at (154.9, 142.2)
- added C3: 10uf, Capacitor_SMD:C_0603_1608Metric, F.Cu at (156.6, 144.7)
- added C4: 2.2uF, Capacitor_SMD:C_0603_1608Metric, F.Cu at (168.0, 131.7)
- added C5: 4u7, Capacitor_SMD:C_0603_1608Metric, F.Cu at (151.3, 147.2)
- added C6: 100nF, Capacitor_SMD:C_0603_1608Metric, F.Cu at (158.9, 142.2)
- added C7: 100n, Capacitor_SMD:C_0603_1608Metric, F.Cu at (152.6, 144.7)
- added C8: 100n, Capacitor_SMD:C_0603_1608Metric, F.Cu at (161.9, 137.7)
- added C9: 100n, Capacitor_SMD:C_0603_1608Metric, F.Cu at (168.0, 129.2)
- added D1: RED, LED_SMD:LED_0201_0603Metric_Castellated, F.Cu at (171.8, 128.9)
- added D2: GREEN, LED_SMD:LED_0201_0603Metric_Castellated, F.Cu at (171.8, 130.8)
- added F1: 500mA, Fuse:Fuse_0805_2012Metric_Castellated, F.Cu at (168.4, 126.5)
- added FB1: ~, Fuse:Fuse_0805_2012Metric, F.Cu at (148.3, 143.9)
- added J1: USB_C_Receptacle_USB2.0, Connector_USB:USB_C_Receptacle_HRO_TYPE-C-31-M-12, F.Cu at (149.2, 79.0)
- added J2: 2199119-4, TE:TE_2199119-4, F.Cu at (149.5, 91.8)
- added L1: 39n, Inductor_SMD:L_0603_1608Metric, F.Cu at (155.3, 147.2)
- added PSW1: TS-1145A-C-B, Button_Switch_SMD:SW_SPST_PTS810, F.Cu at (144.7, 140.1)
- added R1: 1k, Capacitor_SMD:C_0603_1608Metric, F.Cu at (162.9, 140.2)
- added R2: 10k, Capacitor_SMD:C_0603_1608Metric, F.Cu at (160.6, 144.7)
- added R3: 1k, Capacitor_SMD:C_0603_1608Metric, F.Cu at (169.9, 136.8)
- added R4: 1M, Capacitor_SMD:C_0603_1608Metric, F.Cu at (166.9, 140.2)
- added R5: 5.11k, Capacitor_SMD:C_0603_1608Metric, F.Cu at (159.3, 147.2)
- added R6: 5.11k, Capacitor_SMD:C_0603_1608Metric, F.Cu at (164.6, 142.8)
- added U1: MIC5205-3.3YM5, Package_TO_SOT_SMD:SOT-23-5, F.Cu at (143.7, 144.8)
- added U2: STM32F303CCTx, Package_QFP:LQFP-48_7x7mm_P0.5mm, F.Cu at (149.7, 109.0)
- added U3: USBLC6-2SC6, Package_TO_SOT_SMD:SOT-23-6, F.Cu at (150.5, 140.0)
- added Y1: 16MHz, Crystal:Crystal_SMD_3225-4Pin_3.2x2.5mm, F.Cu at (157.3, 138.7)
